File: keynergy_schem.kicad_pcb (KiCad board)
At the start: 2 copper layers, 44 parts, among them J1 Conn_01x03_Pin, J2 Coils, J3 Columns, J3 Conn_01x04_Pin, J4 Conn_01x04_Pin, J5 Conn_01x04_Pin, J6 Conn_01x03_Pin, J7 Conn_01x04_Pin, J8 Conn_01x03_Pin

Commit message: new
Parts:
- removed the J3 at (46.5, 112.5)
- removed the J3 at (331.5, 218.0)
- removed the J3 at (214.5, 287.5)
- added J4: Conn_01x03_Pin, Connector_PinHeader_2.54mm:PinHeader_1x03_P2.54mm_Vertical, F.Cu at (26.7, 82.2)
- added J5: Conn_01x02_Pin, Connector_PinHeader_2.54mm:PinHeader_1x02_P2.54mm_Vertical, F.Cu at (214.5, 287.8)
- added J7: Conn_01x02_Pin, Connector_PinHeader_2.54mm:PinHeader_1x02_P2.54mm_Vertical, F.Cu at (331.5, 217.8)
- J2: value Coils -> Conn_01x03_Pin
- J3: value Columns -> Conn_01x04_Pin
- J4: value Conn_01x04_Pin -> Conn_01x03_Pin; footprint Connector_PinHeader_2.54mm:PinHeader_1x04_P2.54mm_Vertical -> Connector_PinHeader_2.54mm:PinHeader_1x03_P2.54mm_Vertical
- J5, J7: value Conn_01x04_Pin -> Conn_01x02_Pin; footprint Connector_PinHeader_2.54mm:PinHeader_1x04_P2.54mm_Vertical -> Connector_PinHeader_2.54mm:PinHeader_1x02_P2.54mm_Vertical
- moved K5 36.8 mm to (60.0, 62.2)
- moved D5 36.1 mm to (72.8, 80.6)
- moved D6 36.1 mm to (129.8, 79.6)
- moved D7 36.1 mm to (185.3, 79.1)
- moved J2 36.1 mm to (203.3, 29.8)
- moved J4 36.1 mm to (31.8, 82.2)
- moved Jumper 36.1 mm to (172.8, 80.3)
- moved K7 36.1 mm to (172.8, 61.7)
- moved Jumper 36.1 mm to (116.8, 80.8)
- moved K6 36.1 mm to (116.8, 62.2)
Routing:
- net Col 5-3: track 5.66 -> 0.00 mm
- net Col 5-4: track 5.66 -> 0.00 mm
- net Col 2-4: track 5.02 -> 0.00 mm
- net Coil 2-2: track 152.4 -> 151.1 mm
- net Col 2-1: track 37.9 -> 36.9 mm
- net Col 1-4: track 207.0 -> 207.9 mm
Other:
- board outline added: 200.9 x 87.9 mm

Commit message: new
Connections:
- J7 pad 1: (no net) -> Row 5-1
- J7 pad 2: (no net) -> Row 5-2
Routing:
- net Coil 5-4: track 109.4 -> 105.6 mm

Commit message: new update
Other:
- board size 200.9 x 87.9 mm -> 566.2 x 351.8 mm
Changed lines of the file:
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@@
+	)
+	(gr_rect
+		(start 315.341 -36.957)
+		(end 585.216 52.324)
+		(stroke
+			(width 0.05)
+			(type default)
+		)
+		(fill no)
+		(layer "Edge.Cuts")
+	)
+	(gr_rect
+		(start 322.58 61.976)
+		(end 383.794 223.012)
+		(stroke
+			(width 0.05)
+			(type default)
+		)
+		(fill no)
+		(layer "Edge.Cuts")
+	)
+	(gr_rect
+		(start 205.486 225.806)
+		(end 399.796 314.833)
+		(stroke
+			(width 0.05)
+			(type default)
+		)
+		(fill no)
+		(layer "Edge.Cuts")
 	)
 	(gr_rect

Commit message: new updates
Parts:
- moved K7 2.26 mm to (172.0, 59.6)
- moved K6 1.98 mm to (116.8, 60.2)
- moved K5 0.48 mm to (59.7, 61.8)
Routing:
- net Col 2-3: track 152.1 -> 158.4 mm
- net Col 2-2: track 94.9 -> 99.8 mm
- net Col 2-1: track 36.9 -> 40.2 mm
- net Net-(D7-A): track 12.7 -> 15.2 mm
- net Net-(D6-A): track 13.2 -> 15.0 mm
- net Net-(D5-A): track 12.6 -> 11.1 mm
- net Coil 2-2: track 151.1 -> 152.1 mm
Other:
- board size 566.2 x 351.8 mm -> 569.8 x 351.8 mm

Commit message: new updates
Parts:
- moved K7 2.25 mm to (171.3, 61.7)
- moved K6 1.84 mm to (116.1, 61.9)
Routing:
- net Net-(D7-A): track 15.2 -> 11.1 mm
- net Net-(K6-C2): track 58.1 -> 54.3 mm
- net Coil 2-1: track 45.0 -> 48.7 mm
- net Col 2-3: track 158.4 -> 154.7 mm
- net Net-(D6-A): track 15.0 -> 11.9 mm
- net Col 2-2: track 99.8 -> 98.4 mm
- net Net-(K5-C2): track 58.6 -> 57.3 mm
- net Row 2: track 189.1 -> 190.1 mm
Other:
- board size 569.8 x 351.8 mm -> 585.5 x 351.8 mm

Commit message: new
Parts:
- moved K8 89.4 mm to (185.7, 263.7)
- moved K9 88.6 mm to (271.5, 263.4)
- moved D8 87.9 mm to (200.1, 283.3)
- moved D9 87.9 mm to (284.6, 283.3)
- moved J5 87.9 mm to (126.6, 285.8)
- moved J5 87.9 mm to (132.1, 285.7)
- moved J6 87.9 mm to (302.7, 232.0)
- moved Jumper 87.9 mm to (272.1, 284.0)
- moved K1 3.18 mm to (356.1, 6.86)
- moved K2 2.16 mm to (414.3, 6.86)
- moved K11 2.08 mm to (354.8, 116.6)
- moved K3 1.73 mm to (469.9, 6.86)
- moved K10 1.26 mm to (354.1, 184.2)
- moved K4 1.25 mm to (525.3, 6.86)
- moved Jumper 0.89 mm to (334.0, 196.4)
Routing:
- net Net-(D11-A): track 0.00 -> 7.84 mm
- net Col 5-2: track 150.3 -> 157.2 mm
- net Col 1-2: track 94.4 -> 99.8 mm
- net Col 1-3: track 151.3 -> 156.7 mm
- net Col 1-1: track 37.5 -> 42.6 mm
- net Net-(K10-C2): track 79.0 -> 75.2 mm
- net Net-(D1-A): track 13.7 -> 17.3 mm
- net Net-(D8-A): track 13.1 -> 15.9 mm
- net Net-(D2-A): track 13.2 -> 11.0 mm
- net Net-(D9-A): track 12.6 -> 14.7 mm
- net Col 5-1: track 65.3 -> 67.3 mm
- net Net-(D3-A): track 13.0 -> 14.7 mm
- net Net-(K2-C2): track 58.1 -> 57.5 mm
- net Net-(D10-A): track 10.7 -> 11.2 mm
Other:
- board size 585.5 x 351.8 mm -> 585.5 x 349.8 mm

Commit message: new
Parts:
- removed D10, D11, D5, D6, D7, D8, D9: D, Diode_THT:D_DO-35_SOD27_P7.62mm_Horizontal
- removed J2, J4 (x2), J6, J8: Conn_01x03_Pin, Connector_PinHeader_2.54mm:PinHeader_1x03_P2.54mm_Vertical
- removed the J3 at (325.0, 29.5)
- removed the J3 at (331.0, 29.5)
- removed J5 (x2), J7 (x2): Conn_01x02_Pin, Connector_PinHeader_2.54mm:PinHeader_1x02_P2.54mm_Vertical
- removed Jumper (x10): SolderWire-0.1sqmm_1x01_D0.4mm_OD1mm_Relief, Connector_Wire:SolderWire-0.1sqmm_1x01_D0.4mm_OD1mm_Relief
- added A2: RaspberryPi_Pico_W, Module:RaspberryPi_Pico_Common_THT, F.Cu at (527.2, 58.0)
- added C1: 1000uF, Capacitor_THT:CP_Radial_D8.0mm_P5.00mm, F.Cu at (520.6, 146.8)
- added C2: C_Polarized_Small, Capacitor_THT:CP_Radial_D8.0mm_P3.50mm, F.Cu at (521.3, 156.3)
- added D12: D, Diode_THT:D_DO-34_SOD68_P7.62mm_Horizontal, F.Cu at (529.4, 143.6)
- added D13: D, Diode_THT:D_DO-34_SOD68_P7.62mm_Horizontal, F.Cu at (529.4, 146.7)
- added D14: 1N5819, Diode_THT:D_DO-34_SOD68_P7.62mm_Horizontal, F.Cu at (529.4, 149.8)
- added D15: D, Diode_THT:D_DO-34_SOD68_P7.62mm_Horizontal, F.Cu at (529.4, 153.0)
- added J3: Conn_01x04_Pin, Connector_PinHeader_2.54mm:PinHeader_1x04_P2.54mm_Vertical, F.Cu at (34.0, 119.3)
- added K12: ~, project library:Solenoid Key, F.Cu at (-222.3, 256.5)
- added K13: ~, project library:Solenoid Key, F.Cu at (-158.2, 73.2)
- added K14: ~, project library:Solenoid Key, F.Cu at (-158.2, 134.3)
- added K15: ~, project library:Solenoid Key, F.Cu at (-158.2, 195.4)
- added K16: ~, project library:Solenoid Key, F.Cu at (-158.2, 256.5)
- added K17: ~, project library:Solenoid Key, F.Cu at (-94.1, 73.2)
- added K18: ~, project library:Solenoid Key, F.Cu at (-94.1, 134.3)
- added K19: ~, project library:Solenoid Key, F.Cu at (-94.1, 195.4)
- added K20: ~, project library:Solenoid Key, F.Cu at (-94.1, 256.5)
- added R1: 10k, Resistor_THT:R_Axial_DIN0204_L3.6mm_D1.6mm_P7.62mm_Horizontal, F.Cu at (531.1, 166.3)
- added R2: 10k, Resistor_THT:R_Axial_DIN0204_L3.6mm_D1.6mm_P7.62mm_Horizontal, F.Cu at (531.1, 169.4)
- D1, D2, D3, D4: value D -> 1N5818; footprint Diode_THT:D_DO-35_SOD27_P7.62mm_Horizontal -> Diode_THT:D_DO-34_SOD68_P7.62mm_Horizontal
- moved K11 582.5 mm to (-222.3, 195.4), turned to 0 degrees
- moved K10 578.6 mm to (-222.3, 134.3), turned to 0 degrees
- moved K9 529.2 mm to (-222.3, 73.2), turned to 0 degrees
- moved K1 305.8 mm to (60.2, 84.3)
- moved K2 294.2 mm to (130.5, 84.3)
- moved K3 280.3 mm to (200.6, 84.3)
- moved K4 267.1 mm to (269.8, 84.6)
- moved D1 209.3 mm to (545.4, 143.3), turned to 0 degrees
- moved J1 194.9 mm to (531.9, 173.3), turned to 0 degrees
- moved D2 168.7 mm to (545.4, 146.5), turned to 0 degrees
- moved D3 138.4 mm to (545.4, 149.6), turned to 0 degrees
- moved D4 127.3 mm to (545.4, 152.8), turned to 0 degrees
- moved K8 111.2 mm to (243.2, 168.4), turned to 90 degrees
- moved K7 107.3 mm to (182.1, 168.4), turned to 90 degrees
- moved K6 106.7 mm to (121.0, 168.4), turned to 90 degrees
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Connections:
- D1 pad 1: Row 1 -> Net-(D1-K)
- D2 pad 1: Row 1 -> Net-(D2-K)
- D2 pad 2: Net-(D2-A) -> Net-(D1-K)
- D3 pad 1: Row 1 -> Net-(D3-K)
- D3 pad 2: Net-(D3-A) -> Net-(D1-A)
- D4 pad 1: Row 1 -> Net-(D2-K)
- D4 pad 2: Net-(D4-A) -> Net-(D3-K)
- K1 pad 3: Net-(D1-A) -> Row 1
- K1 pad 4: Col 1-1 -> Column 1
- K10 pad 1: Coil 5-4 -> Net-(K10-C1)
- K10 pad 3: Net-(D10-A) -> Row 3
- K10 pad 4: Row 5-1 -> Column 2
- K11 pad 2: Coil 5-3 -> Coil 3-1
- K11 pad 3: Net-(D11-A) -> Row 3
- K11 pad 4: Row 5-2 -> Column 3
- K2 pad 3: Net-(D2-A) -> Row 1
- K2 pad 4: Col 1-2 -> Column 2
- K3 pad 3: Net-(D3-A) -> Row 1
- K3 pad 4: Col 1-3 -> Column 3
- K4 pad 3: Net-(D4-A) -> Row 1
- K4 pad 4: Col 1-4 -> Column 4
- K5 pad 3: Net-(D5-A) -> Row 2
- K5 pad 4: Col 2-1 -> Column 1
- K6 pad 3: Net-(D6-A) -> Row 2
- K6 pad 4: Col 2-2 -> Column 2
- K7 pad 2: Coil 2-1 -> Net-(K7-C2)
- K7 pad 3: Net-(D7-A) -> Row 2
- K7 pad 4: Col 2-3 -> Column 3
- K8 pad 1: Coil 5-2 -> Net-(K7-C2)
- K8 pad 2: Net-(K8-C2) -> Coil 2-1
- K8 pad 3: Net-(D8-A) -> Row 2
- K8 pad 4: Col 5-1 -> Column 4
- K9 pad 1: Net-(K8-C2) -> Coil 3-2
- K9 pad 2: Coil 5-1 -> Net-(K10-C1)
- K9 pad 3: Net-(D9-A) -> Row 3
- K9 pad 4: Col 5-2 -> Column 1
Routing:
- net Column 4: track 0.00 -> 243.8 mm
- net Col 1-4: track 207.9 -> 0.00 mm
- net Row 2: track 190.1 -> 0.00 mm
- net Column 3: track 0.00 -> 185.2 mm
- net Row 5: track 161.7 -> 0.00 mm
- net Col 5-2: track 157.2 -> 0.00 mm
- net Col 1-3: track 156.7 -> 0.00 mm
- net Col 2-3: track 154.7 -> 0.00 mm
- net Coil 2-2: track 152.1 -> 0.00 mm
- net Col 5: track 140.6 -> 0.00 mm
- net Coil 5-2: track 124.2 -> 0.00 mm
- net Column 2: track 0.00 -> 108.9 mm
- net Coil 5-4: track 105.6 -> 0.00 mm
- net Row 5-2: track 100.6 -> 0.00 mm
- net Col 1-2: track 99.8 -> 0.00 mm
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Other:
- board size 585.5 x 349.8 mm -> 9 x 9 mm
- board text removed: "Addition"
- board text removed: "Col 1"
- board text removed: "Col 1-2"
- board text removed: "Col 2"
- board text removed: "Col 3"
- board text removed: "Col 4"
- board text removed: "Col 4-1"
- board text removed: "Col 4-2"
- board text removed: "Division"
- board text removed: "Eight Five Two"
- board text removed: "Enter"
- board text removed: "Multiplication"
- board text removed: "Nine Six Three"
- board text removed: "Num Lock"
- board text removed: "Period"
- board text removed: "Row 1"
- board text removed: "Row 2-4"
- board text removed: "Row 5"
- board text removed: "Seven Four One"
- board text removed: "Subtraction"
- board text removed: "Zero"

Commit message: new update
Parts:
- added J2: Conn_01x04_Pin, Connector_PinHeader_2.54mm:PinHeader_1x04_P2.54mm_Vertical, F.Cu at (162.1, 188.8)
- added J4: Conn_01x04_Pin, Connector_PinHeader_2.54mm:PinHeader_1x04_P2.54mm_Vertical, F.Cu at (285.0, 122.4)
- added J5: Conn_01x04_Pin, Connector_PinHeader_2.54mm:PinHeader_1x04_P2.54mm_Vertical, F.Cu at (162.1, 123.4)
- added J6: Conn_01x04_Pin, Connector_PinHeader_2.54mm:PinHeader_1x04_P2.54mm_Vertical, F.Cu at (162.1, 193.5)
- J1: value Conn_01x03_Pin -> Conn_01x04_Pin; footprint Connector_PinHeader_2.54mm:PinHeader_1x03_P2.54mm_Vertical -> Connector_PinHeader_2.54mm:PinHeader_1x04_P2.54mm_Vertical
- J3: value Conn_01x04_Pin -> Conn_01x02_Pin; footprint Connector_PinHeader_2.54mm:PinHeader_1x04_P2.54mm_Vertical -> Connector_PinHeader_2.54mm:PinHeader_1x02_P2.54mm_Vertical
- moved J1 372.6 mm to (162.1, 127.7), turned to 90 degrees
- moved K12 161.2 mm to (-246.6, 97.1), turned to -90 degrees
- moved K9 160.9 mm to (-63.3, 97.1), turned to -90 degrees
- moved K20 155.6 mm to (-246.6, 225.3), turned to -90 degrees
- moved K17 155.2 mm to (-63.3, 225.3), turned to -90 degrees
- moved K16 129.9 mm to (-246.6, 161.2), turned to -90 degrees
- moved K13 129.5 mm to (-63.3, 161.2), turned to -90 degrees
- moved K11 105.0 mm to (-185.5, 97.1), turned to -90 degrees
- moved K10 104.8 mm to (-124.4, 97.1), turned to -90 degrees
- moved K19 96.1 mm to (-185.5, 225.3), turned to -90 degrees
- moved K18 95.9 mm to (-124.4, 225.3), turned to -90 degrees
- moved K15 43.7 mm to (-185.5, 161.2), turned to -90 degrees
- moved K14 43.3 mm to (-124.4, 161.2), turned to -90 degrees
- moved K8 29.0 mm to (270.4, 158.5), turned to -90 degrees
- moved K7 20.8 mm to (200.3, 158.5), turned to -90 degrees
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Connections:
- J1 pad 1: Row 1 -> Column 1
- J1 pad 2: Coil 1-1 -> Column 2
- J1 pad 3: Coil 1-2 -> Column 3
- J3 pad 1: Column 1 -> Row 1
- J3 pad 2: Column 2 -> Row 2
Routing:
- net Column 1: track 43.5 -> 299.8 mm
- net Row 2: track 0.00 -> 255.7 mm
- net Coil 2-2: track 0.00 -> 232.2 mm
- net Net-(K5-C2): track 0.00 -> 72.1 mm
- net Net-(K7-C2): track 0.00 -> 71.8 mm
- net Net-(K6-C2): track 0.00 -> 71.7 mm
- net Column 2: track 108.9 -> 177.4 mm
- net Column 4: track 243.8 -> 295.9 mm
- net Coil 2-1: track 0.00 -> 30.0 mm
- net Row 1: track 262.4 -> 250.5 mm
- net Column 3: track 185.2 -> 174.5 mm
- net Coil 1-1: track 67.9 -> 61.6 mm
- net Net-(K2-C2): track 65.7 -> 70.2 mm
- net Coil 1-2: track 282.9 -> 280.3 mm
- net Net-(K3-C2): track 69.7 -> 71.9 mm
