File: keynergy_schem.kicad_pcb (KiCad board)
At the start: 2 copper layers, 9 x 9 mm, 39 parts, among them J1 Conn_01x04_Pin, J2 Conn_01x04_Pin, J3 Conn_01x02_Pin, J4 Conn_01x04_Pin, J5 Conn_01x04_Pin, J6 Conn_01x04_Pin

Commit message: new updates
Parts:
- moved K9 370.1 mm to (270.4, 257.3)
- moved K10 362.1 mm to (200.4, 257.3)
- moved K11 354.2 mm to (130.4, 257.3)
- moved K13 349.1 mm to (243.5, 327.9)
- moved K14 349.1 mm to (182.4, 327.9)
- moved K15 349.1 mm to (121.3, 327.9)
- moved K16 349.1 mm to (60.2, 327.9)
- moved K12 345.8 mm to (59.9, 257.3)
Changed lines of the file:
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@@
 	(footprint "project library:Solenoid Key"
 		(layer "F.Cu")
-		(at -246.5615 97.136 -90)
+		(at 59.9 257.335 -90)
 		(property "Reference" "K12"
 			(at -1.016 -0.5 270)
@@
 	(footprint "project library:Solenoid Key"
 		(layer "F.Cu")
-		(at -63.2615 97.136 -90)
+		(at 270.4 257.271 -90)
 		(property "Reference" "K9"
 			(at -1.016 -0.5 270)
@@
 	(footprint "project library:Solenoid Key"
 		(layer "F.Cu")
-		(at -124.3615 161.236 -90)
+		(at 182.4 327.935 -90)
 		(property "Reference" "K14"
 			(at -1.016 -0.5 270)
@@
 	(footprint "project library:Solenoid Key"
 		(layer "F.Cu")
-		(at -185.4615 97.136 -90)
+		(at 130.4 257.335 -90)
 		(property "Reference" "K11"
 			(at -1.016 -0.5 270)
@@
 	(footprint "project library:Solenoid Key"
 		(layer "F.Cu")
-		(at -63.2615 161.236 -90)
+		(at 243.5 327.935 -90)
 		(property "Reference" "K13"
 			(at -1.016 -0.5 270)
@@
 	(footprint "project library:Solenoid Key"
 		(layer "F.Cu")
-		(at -124.3615 97.136 -90)
+		(at 200.4 257.335 -90)
 		(property "Reference" "K10"
 			(at -1.016 -0.5 270)
@@
 	(footprint "project library:Solenoid Key"
 		(layer "F.Cu")
-		(at -185.4615 161.236 -90)
+		(at 121.3 327.935 -90)
 		(property "Reference" "K15"
 			(at -1.016 -0.5 270)
@@
 	(footprint "project library:Solenoid Key"
 		(layer "F.Cu")
-		(at -246.5615 161.236 -90)
+		(at 60.2 327.935 -90)
 		(property "Reference" "K16"
 			(at -1.016 -0.5 270)
@@
 	)
 	(segment
+		(start 50 127.94)
+		(end 50 132)
+		(width 2)
+		(layer "F.Cu")
+		(net 49)
+	)
+	(segment
 		(start 207.351 165.726)
 		(end 207.451 165.826)
@@
 	)
 	(segment
-		(start 50 127.94)
-		(end 50 161.4895)
+		(start 50 132)
+		(end 52 134)
 		(width 2)
 		(layer "F.Cu")
@@
 	)
 	(segment
-		(start 50 161.4895)
-		(end 54.2365 165.726)
+		(start 52 134)
+		(end 52 163.4895)
 		(width 2)
 		(layer "F.Cu")
@@
 	)
 	(segment
+		(start 52 163.4895)
+		(end 54.2365 165.726)
+		(width 2)
+		(layer "F.Cu")
+		(net 49)
+	)
+	(segment
 		(start 54.2365 165.726)
 		(end 59.9865 165.726)
@@
 	)
 	(segment
-		(start 50 96.8375)
+		(start 52 94.8375)
+		(end 52 119)
+		(width 2)
+		(layer "F.Cu")
+		(net 76)
+	)
+	(segment
+		(start 50 121)
 		(end 50 125)
 		(width 2)
@@
 	)
 	(segment
-		(start 54.2865 92.551)
-		(end 50 96.8375)
+		(start 152.551 92.551)
+		(end 152.786 92.786)
 		(width 2)
 		(layer "F.Cu")
@@
 	)
 	(segment
-		(start 152.551 92.551)
-		(end 152.786 92.786)
+		(start 54.2865 92.551)
+		(end 52 94.8375)
 		(width 2)
 		(layer "F.Cu")
@@
 		(width 2)
 		(layer "F.Cu")
+		(net 76)
+	)
+	(segment
+		(start 52 119)
+		(end 50 121)
+		(width 2)
+		(layer "F.Cu")

Commit message: new updates, pdf exported
Parts:
- added J7: Conn_01x04_Pin, Connector_PinHeader_2.54mm:PinHeader_1x04_P2.54mm_Vertical, F.Cu at (-32.6, 148.8)
- added J8: Conn_01x04_Pin, Connector_PinHeader_2.54mm:PinHeader_1x04_P2.54mm_Vertical, F.Cu at (214.6, 161.6)
- added REF**: MountingHole_3.2mm_M3_Pad, MountingHole:MountingHole_3.2mm_M3_Pad, F.Cu at (112.8, 93.3)
- added REF**: MountingHole_3.2mm_M3_Pad, MountingHole:MountingHole_3.2mm_M3_Pad, F.Cu at (183.0, 93.3)
- added REF**: MountingHole_3.2mm_M3_Pad, MountingHole:MountingHole_3.2mm_M3_Pad, F.Cu at (148.6, 23.9)
- moved A2 718.3 mm to (-190.6, 30.3)
- moved C1 718.3 mm to (-197.2, 119.0)
- moved C2 718.3 mm to (-196.4, 128.5)
- moved D1 718.3 mm to (-172.4, 115.6)
- moved D12 718.3 mm to (-188.4, 115.8)
- moved D13 718.3 mm to (-188.4, 118.9)
- moved D14 718.3 mm to (-188.4, 122.1)
- moved D15 718.3 mm to (-188.4, 125.2)
- moved D2 718.3 mm to (-172.4, 118.7)
- moved D3 718.3 mm to (-172.4, 121.9)
- moved D4 718.3 mm to (-172.4, 125.0)
- moved R1 718.3 mm to (-186.7, 138.5)
- moved R2 718.3 mm to (-186.7, 141.7)
- moved K10 350.0 mm to (-142.6, 326.7)
- moved K11 350.0 mm to (-212.6, 326.7)
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Connections:
- J4 pad 1: Coil 1-2 -> Coil 1-1
- J4 pad 2: Coil 1-1 -> Coil 1-2
Routing:
- net Coil 1-2: track 280.3 -> 390.2 mm
- net Coil 2-1: track 30.0 -> 137.0 mm
- net Coil 1-1: track 61.6 -> 163.9 mm
- net Coil 2-2: track 232.2 -> 256.5 mm
- net Row 2: track 255.7 -> 258.8 mm
- net (no net): vias 0 -> 1
Other:
- board text added: "C1"
- board text added: "C2"
- board text added: "Col1"
- board text added: "Col2"
- board text added: "Col3"
- board text added: "Col4"
- board text added: "ROW"
- board text added: "TOP"
- board text added: "^^^ J1"
- board text added: "^^^ J2"
- board text added: "^^^ J6"

Commit message: new updates
Parts:
- removed K10, K11, K12, K13, K14, K15, K16, K9: ~, project library:Solenoid Key
- added J1: Conn_01x04_Pin, Connector_PinHeader_2.54mm:PinHeader_1x04_P2.54mm_Vertical, F.Cu at (144.8, 131.1)
- added J1: Conn_01x04_Pin, Connector_PinHeader_2.54mm:PinHeader_1x04_P2.54mm_Vertical, F.Cu at (144.8, 67.6)
- added J3: Conn_01x02_Pin, Connector_PinHeader_2.54mm:PinHeader_1x02_P2.54mm_Vertical, F.Cu at (38.5, 124.1)
- added J4: Conn_01x04_Pin, Connector_PinHeader_2.54mm:PinHeader_1x04_P2.54mm_Vertical, F.Cu at (214.7, 67.1)
- added J4: Conn_01x04_Pin, Connector_PinHeader_2.54mm:PinHeader_1x04_P2.54mm_Vertical, F.Cu at (228.3, 128.1)
- added J5: Conn_01x04_Pin, Connector_PinHeader_2.54mm:PinHeader_1x04_P2.54mm_Vertical, F.Cu at (144.8, 127.1)
- added J9: Conn_01x04_Pin, Connector_PinHeader_2.54mm:PinHeader_1x04_P2.54mm_Vertical, F.Cu at (214.8, 128.1)
- added REF**: MountingHole_3.2mm_M3_Pad, MountingHole:MountingHole_3.2mm_M3_Pad, F.Cu at (183.1, 130.1)
- added REF**: MountingHole_3.2mm_M3_Pad, MountingHole:MountingHole_3.2mm_M3_Pad, F.Cu at (112.1, 130.1)
- added REF**: MountingHole_3.2mm_M3_Pad, MountingHole:MountingHole_3.2mm_M3_Pad, F.Cu at (268.1, 67.1)
- moved K20 517.4 mm to (253.2, 91.5)
- moved K19 392.2 mm to (183.1, 91.2)
- moved J7 390.7 mm to (-418.2, 212.2)
- moved K1 370.9 mm to (-290.3, 216.7)
- moved J1 370.9 mm to (-188.3, 259.3)
- moved J2 370.9 mm to (-188.3, 320.4)
- moved J3 370.9 mm to (-300.3, 256.6)
- moved J4 370.9 mm to (-118.3, 257.3)
- moved J5 370.9 mm to (-188.3, 255.0)
- moved J6 370.9 mm to (-188.3, 325.1)
- moved K2 370.9 mm to (-220.0, 216.7)
- moved K3 370.9 mm to (-150.0, 216.7)
- moved K6 370.9 mm to (-220.0, 290.0)
- moved K7 370.9 mm to (-150.0, 290.0)
- moved K8 370.9 mm to (-79.9, 290.0)
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Connections:
- K17 pad 1: Coil 5-2 -> Coil 1-2
- K17 pad 2: Net-(K17-C2) -> Net-(K1-C2)
- K17 pad 3: Row 5 -> Row 1
- K18 pad 1: Net-(K17-C2) -> Net-(K1-C2)
- K18 pad 2: Net-(K18-C2) -> Net-(K2-C2)
- K18 pad 3: Row 5 -> Row 1
- K19 pad 1: Net-(K18-C2) -> Net-(K2-C2)
- K19 pad 2: Coil 5-1 -> Net-(K3-C2)
- K19 pad 3: Row 5 -> Row 1
- K20 pad 1: unconnected-(K20-C1-Pad1) -> Net-(K3-C2)
- K20 pad 2: unconnected-(K20-C2-Pad2) -> Coil 1-1
- K20 pad 3: Row 5 -> Row 1
Routing:
- net Coil 1-2: track 390.2 -> 730.4 mm
- net Row 1: track 250.5 -> 498.7 mm
- net Column 1: track 299.8 -> 476.0 mm
- net Column 4: track 295.9 -> 470.7 mm
- net Coil 1-1: track 163.9 -> 285.3 mm
- net Column 2: track 177.3 -> 295.4 mm
- net Column 3: track 174.5 -> 290.8 mm
- net Net-(K1-C2): track 73.7 -> 147.4 mm
- net Net-(K3-C2): track 71.9 -> 143.8 mm
- net Net-(K2-C2): track 70.2 -> 140.5 mm
- net Coil 2-2: track 256.5 -> 253.6 mm
- net Coil 2-1: track 137.0 -> 134.1 mm

Commit message: updated
Parts:
- added J1: Conn_01x04_Pin, Connector_PinHeader_2.54mm:PinHeader_1x04_P2.54mm_Vertical, F.Cu at (144.8, 67.9)
- moved J7 386.8 mm to (-39.9, 131.6)
- moved J1 4.83 mm to (144.9, 72.4)
Routing:
- net Coil 1-2: track 730.4 -> 732.4 mm

Commit message: new
Parts:
- removed A2: RaspberryPi_Pico_W, Module:RaspberryPi_Pico_Common_THT
- removed C1: 1000uF, Capacitor_THT:CP_Radial_D8.0mm_P5.00mm
- removed C2: C_Polarized_Small, Capacitor_THT:CP_Radial_D8.0mm_P3.50mm
- removed D1, D2, D3, D4: 1N5818, Diode_THT:D_DO-34_SOD68_P7.62mm_Horizontal
- removed D13, D15: D, Diode_THT:D_DO-34_SOD68_P7.62mm_Horizontal
- removed D14: 1N5819, Diode_THT:D_DO-34_SOD68_P7.62mm_Horizontal
- removed J7: Conn_01x04_Pin, Connector_PinHeader_2.54mm:PinHeader_1x04_P2.54mm_Vertical
- removed R1, R2: 10k, Resistor_THT:R_Axial_DIN0204_L3.6mm_D1.6mm_P7.62mm_Horizontal
- added D10: 1N4001, Diode_THT:D_DO-34_SOD68_P7.62mm_Horizontal, F.Cu at (-203.4, 273.1)
- added D11: 1N4001, Diode_THT:D_DO-34_SOD68_P7.62mm_Horizontal, F.Cu at (-134.2, 273.1)
- added D5: 1N4001, Diode_THT:D_DO-34_SOD68_P7.62mm_Horizontal, F.Cu at (-279.4, 199.6)
- added D6: 1N4001, Diode_THT:D_DO-34_SOD68_P7.62mm_Horizontal, F.Cu at (-207.6, 199.9)
- added D7: 1N4001, Diode_THT:D_DO-34_SOD68_P7.62mm_Horizontal, F.Cu at (-159.1, 199.6)
- added D8: 1N4001, Diode_THT:D_DO-34_SOD68_P7.62mm_Horizontal, F.Cu at (-90.9, 200.1)
- added D9: 1N4001, Diode_THT:D_DO-34_SOD68_P7.62mm_Horizontal, F.Cu at (-263.4, 273.0)
- added J4: Conn_01x04_Pin, Connector_PinHeader_2.54mm:PinHeader_1x04_P2.54mm_Vertical, F.Cu at (-118.3, 260.3)
- added J8: Conn_01x04_Pin, Connector_PinHeader_2.54mm:PinHeader_1x04_P2.54mm_Vertical, F.Cu at (-118.2, 321.0)
- D12: value D -> 1N4001
- moved D12 183.9 mm to (-93.2, 273.1), turned to -90 degrees
- moved J8 5.24 mm to (-118.3, 317.1)
- moved J6 2.51 mm to (-188.2, 322.6)
- moved J2 1.71 mm to (-188.2, 318.6)
Connections:
- D12 pad 1: IN+ -> Coil 2-2
- D12 pad 2: Combined Coil 1 -> Net-(D12-A)
- J3 pad 2: Row 1 -> Row 2
- J4 pad 1: (no net) -> Coil 1-1
- J4 pad 2: (no net) -> Coil 1-2
- J4 pad 3: (no net) -> Coil 2-2
- J4 pad 4: (no net) -> Coil 2-1
- J4 pad 3: Coil 1-1 -> Coil 2-2
- J4 pad 4: Coil 1-2 -> Coil 2-1
- K1 pad 1: Coil 1-2 -> Coil 1-1
- K1 pad 2: Net-(K1-C2) -> Net-(D5-A)
- K2 pad 1: Net-(K1-C2) -> Coil 1-1
- K2 pad 2: Net-(K2-C2) -> Net-(D6-A)
- K3 pad 1: Net-(K2-C2) -> Coil 1-1
- K3 pad 2: Net-(K3-C2) -> Net-(D7-A)
- K4 pad 1: Net-(K3-C2) -> Coil 1-1
- K4 pad 2: Coil 1-1 -> Net-(D8-A)
- K5 pad 1: Coil 2-2 -> Coil 2-1
- K5 pad 2: Net-(K5-C2) -> Net-(D9-A)
- K6 pad 1: Net-(K5-C2) -> Coil 2-1
- K6 pad 2: Net-(K6-C2) -> Net-(D10-A)
- K7 pad 1: Net-(K6-C2) -> Coil 2-1
- K7 pad 2: Net-(K7-C2) -> Net-(D11-A)
- K8 pad 1: Net-(K7-C2) -> Coil 2-1
- K8 pad 2: Coil 2-1 -> Net-(D12-A)
Routing:
- net Coil 1-1: track 285.3 -> 508.2 mm
- net Coil 2-1: track 134.1 -> 320.0 mm
- net Net-(K1-C2): track 147.4 -> 73.7 mm
- net Net-(K5-C2): track 72.1 -> 0.00 mm
- net Net-(K3-C2): track 143.8 -> 71.9 mm
- net Net-(K7-C2): track 71.8 -> 0.00 mm
- net Net-(K6-C2): track 71.7 -> 0.00 mm
- net Net-(K2-C2): track 140.5 -> 70.2 mm
- net Net-(D9-A): track 0.00 -> 27.0 mm
- net Coil 2-2: track 253.6 -> 278.2 mm
- net Net-(D10-A): track 0.00 -> 16.6 mm
- net Net-(D11-A): track 0.00 -> 15.8 mm
- net Net-(D12-A): track 0.00 -> 13.3 mm
- net Net-(D6-A): track 0.00 -> 12.4 mm
- net Net-(D8-A): track 0.00 -> 11.0 mm
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Other:
- board text added: "JMP^"
- board text added: "^JMP^"
- board text removed: "^^^ J2"
- board text removed: "^^^ J6"

Commit message: new
Parts:
- added ?: , , F.Cu at (271.4, 172.9)
- added ?: , , F.Cu at (28.3, 173.4)
- added ?: , , F.Cu at (270.9, 32.6)
- added ?: , , F.Cu at (28.8, 32.1)
- added J3: Conn_01x02_Pin, Connector_PinHeader_2.54mm:PinHeader_1x02_P2.54mm_Vertical, F.Cu at (34.8, 105.6)
- moved D5 377.5 mm to (64.4, 43.5)
- moved D12 369.7 mm to (241.8, 116.9)
- moved D11 369.7 mm to (200.8, 116.9)
- moved D6 369.7 mm to (127.4, 43.7)
- moved D7 369.7 mm to (176.0, 43.4)
- moved D8 369.7 mm to (244.1, 43.9)
- moved J3 369.7 mm to (34.7, 100.3)
- moved J4 369.7 mm to (216.7, 101.1)
- moved J5 369.7 mm to (146.7, 98.8)
- moved J6 369.7 mm to (146.8, 166.3)
- moved J8 369.7 mm to (216.8, 160.9)
- moved J8 369.7 mm to (216.8, 164.8)
- moved K1 369.7 mm to (44.7, 60.5)
- moved K3 369.7 mm to (185.1, 60.5)
- moved D10 369.7 mm to (131.6, 116.9)
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Routing:
- net Coil 1-2: track 743.4 -> 734.0 mm
- net Net-(D5-A): track 11.0 -> 19.7 mm
- net Coil 2-2: track 278.2 -> 286.6 mm
- net Net-(D9-A): track 27.0 -> 19.8 mm
- net Row 1: track 498.7 -> 504.2 mm
- net Row 2: track 261.2 -> 257.2 mm
- net Coil 1-1: track 508.2 -> 505.4 mm
- net Coil 2-1: track 320.0 -> 322.4 mm

Commit message: new
Parts:
- removed the J4 at (-100.7, 95.9)
- removed the J9 at (-114.3, 95.9)
- added D13: 1N4001, Diode_THT:D_DO-34_SOD68_P7.62mm_Horizontal, F.Cu at (53.1, 87.6)
- added D14: 1N4001, Diode_THT:D_DO-34_SOD68_P7.62mm_Horizontal, F.Cu at (123.4, 87.5)
- added D15: 1N4001, Diode_THT:D_DO-34_SOD68_P7.62mm_Horizontal, F.Cu at (193.2, 87.6)
- added D16: 1N4001, Diode_THT:D_DO-34_SOD68_P7.62mm_Horizontal, F.Cu at (237.5, 87.8)
- added J10: Conn_01x04_Pin, Connector_PinHeader_2.54mm:PinHeader_1x04_P2.54mm_Vertical, F.Cu at (221.7, 84.7)
- added J9: Conn_01x02_Pin, Connector_PinHeader_2.54mm:PinHeader_1x02_P2.54mm_Vertical, F.Cu at (214.9, 139.0)
- added J9: Conn_01x02_Pin, Connector_PinHeader_2.54mm:PinHeader_1x02_P2.54mm_Vertical, F.Cu at (214.8, 134.7)
- moved REF** 416.2 mm to (267.9, 143.2)
- moved J10 339.1 mm to (221.7, 80.7), turned to -90 degrees
- moved ? 335.3 mm to (-44.2, 286.4)
- moved D12 335.3 mm to (-73.7, 230.4)
- moved D6 335.3 mm to (-188.1, 157.2)
- moved D8 335.3 mm to (-71.4, 157.4)
- moved J3 335.3 mm to (-280.7, 219.1)
- moved J8 335.3 mm to (-98.7, 278.3)
- moved K1 335.3 mm to (-270.8, 174.0)
- moved ? 335.3 mm to (-287.2, 286.9)
- moved ? 335.3 mm to (-44.7, 146.2)
- moved ? 335.3 mm to (-286.7, 145.6)
- moved D10 335.3 mm to (-183.9, 230.4)
- moved D11 335.3 mm to (-114.7, 230.4)
- moved D5 335.3 mm to (-251.2, 157.0)
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- renumbered J4 to J10, K18 to K10, K19 to K11, K20 to K12, K17 to K9
Connections:
- J10 pad 1: Coil 1-1 -> Coil 2-2
- J10 pad 2: Coil 1-2 -> Coil 2-1
- K10 pad 1: Net-(K1-C2) -> Coil 2-1
- K10 pad 2: Net-(K2-C2) -> Net-(D14-A)
- K10 pad 3: Row 1 -> Row 3
- K11 pad 1: Net-(K2-C2) -> Coil 2-1
- K11 pad 2: Net-(K3-C2) -> Net-(D15-A)
- K11 pad 3: Row 1 -> Row 3
- K12 pad 1: Net-(K3-C2) -> Coil 2-1
- K12 pad 2: Coil 1-1 -> Net-(D16-A)
- K12 pad 3: Row 1 -> Row 3
- K9 pad 1: Coil 1-2 -> Coil 2-1
- K9 pad 2: Net-(K1-C2) -> Net-(D13-A)
- K9 pad 3: Row 1 -> Row 3
Routing:
- net Coil 2-2: track 286.6 -> 695.7 mm
- net Coil 2-1: track 322.4 -> 721.2 mm
- net Coil 1-2: track 734.0 -> 388.9 mm
- net Row 1: track 504.2 -> 256.0 mm
- net Row 3: track 0.00 -> 248.2 mm
- net Coil 1-1: track 505.4 -> 381.1 mm
- net Net-(K1-C2): track 73.7 -> 0.00 mm
- net Net-(K3-C2): track 71.9 -> 0.00 mm
- net Net-(K2-C2): track 70.2 -> 0.00 mm
- net Net-(D16-A): track 0.00 -> 14.6 mm
- net Net-(D13-A): track 0.00 -> 11.8 mm
- net Net-(D14-A): track 0.00 -> 11.5 mm
- net Net-(D15-A): track 0.00 -> 11.2 mm
- net Column 2: track 293.2 -> 283.6 mm
- net Column 3: track 288.5 -> 280.9 mm
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Other:
- board text removed: "^^^ J1"
